File: RF-AMP-CNTLR_V1.kicad_pcb (KiCad board)
At the start: 4 copper layers, 220 x 100 mm, 382 parts, among them J101 VAC, J102 VDC, J103 ext_13V8, J104 Front Panel, J105 ANT_SWITCH, J106 BAND_SELECT, J107 I2C0, J108 VDD_IN, J109 VSS_IN, J110 RELAY RF OUT, J111 RELAY RF IN, J112 FWD3, J113 REF3, J114 FWD4, J115 REF4, J116 PTT, J117 ALC, J118 VDD_AMP, J119 GND_AMP, J120 SPI0, J121 I2C1, J122 RS232, J123 AMP1, J124 AMP2, J201 Raspberry_Pi_2_3, Q101 DTA124E, Q201 BSS138, Q202 BSS138, Q301 BC857, Q302 BC857, Q303 BC857, Q304 BC857, Q305 BC857, Q306 BC857, Q307 BC857, Q308 BC857, Q309 BC857, Q310 BC857, Q311 BC857, Q312 BC857, Q313 DTC124E, Q314 DTC124E, Q315 DTC124E, Q316 DTC124E, Q317 BC857, Q318 BC857, Q319 BC857, Q320 BC857, Q321 DTA124E, Q322 DTA124E, Q323 BC857, Q324 BC857, Q325 DTC124E, Q326 DTC124E, Q327 DTC124E, Q328 DTC124E, Q329 DTC124E, Q330 DTC124E, Q331 DTC124E, Q332 DTA124E, Q401 IXTH140P10T, Q402 IXTH140P10T, Q403 DTC124E, Q404 BC857, Q405 DTC124E, Q406 DTC124E, Q407 DTC124E, Q408 DTA124E, Q409 DTC124E, Q410 DTC124E, Q411 DTA124E, Q412 BCX53, Q413 DTA124E, Q414 DTC124E, Q415 DTC124E, Q416 BCX53, Q417 DTA124E, Q418 DTC124E, Q419 DTC124E, Q420 BCX53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

Commit message: initial commit
Routing:
- net Earth: track 109.6 -> 186.9 mm

Commit message: Review 1
Parts:
- added D103: BAT54CW, Package_TO_SOT_SMD:SOT-323_SC-70, B.Cu at (139.8, 104.0)
- added D104: BAT54CW, Package_TO_SOT_SMD:SOT-323_SC-70, B.Cu at (104.8, 110.5)
- C105: value 470n -> 47u; footprint Capacitor_THT:C_Rect_L7.0mm_W3.5mm_P5.00mm -> Capacitor_Tantalum_SMD:CP_EIA-6032-28_Kemet-C
- C108: value 33n -> 470n
- D401: value SMZ24 -> SMZ33
- R103: value 470k -> 620
- R407: value 1k8 -> 39k
- moved D101 7.62 mm to (27.6, 73.8), turned to 0 degrees
- moved C105 4.95 mm to (30.2, 69.2)
- moved R103 4.60 mm to (36.0, 68.2)
- turned C202 to 90 degrees
Connections:
- net ILK_CMD renamed ILK_CMD_PI
- C109 pad 2: Net-(C108-Pad2) -> Net-(C109-Pad2)
- C202 pad 1: Earth -> +5V
- C202 pad 2: +5V -> Earth
- D101 pad 3: Net-(C103-Pad2) -> Net-(C109-Pad2)
- J104 pad 12: RESET_CMD -> Net-(D104-Pad1)
- J104 pad 16: OP -> Net-(D103-Pad1)
- J201 pad 16: RESET_CMD -> RESET_CMD_PI
- J201 pad 18: OP -> OP_CMD_PI
Routing:
- net Net-(D104-Pad1): track 0.00 -> 43.3 mm, vias 0 -> 1
- net RESET_CMD: track 74.4 -> 38.5 mm, vias 1 -> 2
- net OP_CMD_PI: track 0.00 -> 33.4 mm, vias 0 -> 1
- net Earth: track 186.9 -> 211.1 mm
- net OP: track 145.8 -> 124.2 mm, vias 2 -> 3
- net Net-(C103-Pad2): track 119.9 -> 108.5 mm
- net Net-(C105-Pad2): track 16.0 -> 25.7 mm
- net Net-(C109-Pad2): track 0.00 -> 6.64 mm
- net Net-(C108-Pad2): track 12.4 -> 6.35 mm
- net Net-(D103-Pad1): track 0.00 -> 4.90 mm
- net Net-(R103-Pad2): track 7.82 -> 11.4 mm
- net /CONTROLLER/INT_OC: track 95.7 -> 98.9 mm
- net +12V: track 838.4 -> 835.6 mm
- net RESET_CMD_PI: track 0.00 -> 2.54 mm
- net Net-(C105-Pad1): track 8.39 -> 10.3 mm
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
Commit message: Review 2
Parts:
- D401: value SMZ33 -> Z1SMA33; footprint Diode_SMD:D_MELF -> Diode_SMD:D_SMA
- R407: value 39k -> 4k7
- moved D401 0.76 mm to (216.8, 111.2)
Routing:
- net Earth: track 211.1 -> 213.5 mm
- net /SEQUENCER/VDD_IN: track 15.3 -> 15.9 mm
Other:
- net class Vdd added: clearance 1, trace_width 0.25, via_dia 0.8, via_drill 0.4
Changed lines of the file:
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@@
-(kicad_pcb (version 20171130) (host pcbnew 5.1.4+dfsg1-1~bpo10+1)
+(kicad_pcb (version 20171130) (host pcbnew 5.1.5+dfsg1-2~bpo10+1)
   (general
     (thickness 1.6)
     (drawings 13)
-    (tracks 2530)
+    (tracks 2532)
     (zones 0)
     (modules 384)
@@
     (34 B.Paste user hide)
     (35 F.Paste user hide)
-    (36 B.SilkS user hide)
+    (36 B.SilkS user)
     (37 F.SilkS user)
     (38 B.Mask user hide)
@@
       (plotinvisibletext false)
       (padsonsilk false)
-      (subtractmaskfromsilk true)
+      (subtractmaskfromsilk false)
       (outputformat 1)
       (mirror false)
@@
     (add_net /SEQUENCER/RELAY2)
     (add_net /SEQUENCER/RELAY2_ON)
-    (add_net /SEQUENCER/VDD)
-    (add_net /SEQUENCER/VDD_IN)
     (add_net ALC_EN)
     (add_net ALC_MON)
@@
     (add_net "Net-(F102-Pad2)")
   )
+  (net_class Vdd ""
+    (clearance 1)
+    (trace_width 0.25)
+    (via_dia 0.8)
+    (via_drill 0.4)
+    (uvia_dia 0.3)
+    (uvia_drill 0.1)
+    (add_net /SEQUENCER/VDD)
+    (add_net /SEQUENCER/VDD_IN)
+  )
   (module Symbol:KiCad-Logo2_8mm_SilkScreen (layer F.Cu)
     (at 114 68.8)
@@
     )
   )
-  (module Diode_SMD:D_MELF (layer B.Cu)
-    (at 217.5 111.4 180)
-    (descr "Diode, MELF,,")
-    (tags "Diode MELF ")
-    (attr smd)
-    (fp_text reference D401 (at -5.6 1.4) (layer B.SilkS)
-      (effects (font (size 1 1) (thickness 0.15)) (justify mirror))
-    )
-    (fp_text value SMZ33 (at -0.25 -2.5) (layer B.Fab)
-      (effects (font (size 1 1) (thickness 0.15)) (justify mirror))
-    )
-    (fp_text user %R (at 0 2.5) (layer B.Fab)
-      (effects (font (size 1 1) (thickness 0.15)) (justify mirror))
-    )
-    (fp_line (start 2.4 1.5) (end -3.3 1.5) (layer B.SilkS) (width 0.12))
-    (fp_line (start -3.3 1.5) (end -3.3 -1.5) (layer B.SilkS) (width 0.12))
-    (fp_line (start -3.3 -1.5) (end 2.4 -1.5) (layer B.SilkS) (width 0.12))
-    (fp_line (start 2.6 1.3) (end -2.6 1.3) (layer B.Fab) (width 0.1))
-    (fp_line (start -2.6 1.3) (end -2.6 -1.3) (layer B.Fab) (width 0.1))
-    (fp_line (start -2.6 -1.3) (end 2.6 -1.3) (layer B.Fab) (width 0.1))
-    (fp_line (start 2.6 -1.3) (end 2.6 1.3) (layer B.Fab) (width 0.1))
-    (fp_line (start -0.64944 -0.00102) (end -1.55114 -0.00102) (layer B.Fab) (width 0.1))
-    (fp_line (start 0.50118 -0.00102) (end 1.4994 -0.00102) (layer B.Fab) (width 0.1))
-    (fp_line (start -0.64944 0.79908) (end -0.64944 -0.80112) (layer B.Fab) (width 0.1))
-    (fp_line (start 0.50118 -0.75032) (end 0.50118 0.79908) (layer B.Fab) (width 0.1))
-    (fp_line (start -0.64944 -0.00102) (end 0.50118 -0.75032) (layer B.Fab) (width 0.1))
-    (fp_line (start -0.64944 -0.00102) (end 0.50118 0.79908) (layer B.Fab) (width 0.1))
-    (fp_line (start -3.4 1.6) (end 3.4 1.6) (layer B.CrtYd) (width 0.05))
-    (fp_line (start 3.4 1.6) (end 3.4 -1.6) (layer B.CrtYd) (width 0.05))
-    (fp_line (start 3.4 -1.6) (end -3.4 -1.6) (layer B.CrtYd) (width 0.05))
-    (fp_line (start -3.4 -1.6) (end -3.4 1.6) (layer B.CrtYd) (width 0.05))
-    (pad 1 smd rect (at -2.4 0 180) (size 1.5 2.7) (layers B.Cu B.Paste B.Mask)
-      (net 211 /SEQUENCER/VDD_IN))
-    (pad 2 smd rect (at 2.4 0 180) (size 1.5 2.7) (layers B.Cu B.Paste B.Mask)
-      (net 213 /SEQUENCER/INA_GND))
-    (model ${KISYS3DMOD}/Diode_SMD.3dshapes/D_MELF.wrl
-      (at (xyz 0 0 0))
-      (scale (xyz 1 1 1))
-      (rotate (xyz 0 0 0))
-    )
-  )
   (module Diode_SMD:D_SOD-523 (layer F.Cu)
     (at 160.3 72.5)
@@
       (effects (font (size 1 1) (thickness 0.15)) (justify mirror))
     )
-    (fp_text value 39k (at 0 -1.65 270) (layer B.Fab)
+    (fp_text value 4k7 (at 0 -1.65 270) (layer B.Fab)
       (effects (font (size 1 1) (thickness 0.15)) (justify mirror))
     )
@@
     )
   )
+  (module Diode_SMD:D_SMA (layer B.Cu)
+    (at 216.75 111.25 180)
+    (descr "Diode SMA (DO-214AC)")
+    (tags "Diode SMA (DO-214AC)")
+    (attr smd)
+    (fp_text reference D401 (at -5.5 -0.75) (layer B.SilkS)
+      (effects (font (size 1 1) (thickness 0.15)) (justify mirror))
+    )
+    (fp_text value Z1SMA33 (at 0 -2.6) (layer B.Fab)
+      (effects (font (size 1 1) (thickness 0.15)) (justify mirror))
+    )
+    (fp_text user %R (at 0 2.5) (layer B.Fab)
+      (effects (font (size 1 1) (thickness 0.15)) (justify mirror))
+    )
+    (fp_line (start -3.4 1.65) (end -3.4 -1.65) (layer B.SilkS) (width 0.12))
+    (fp_line (start 2.3 -1.5) (end -2.3 -1.5) (layer B.Fab) (width 0.1))
+    (fp_line (start -2.3 -1.5) (end -2.3 1.5) (layer B.Fab) (width 0.1))
+    (fp_line (start 2.3 1.5) (end 2.3 -1.5) (layer B.Fab) (width 0.1))
+    (fp_line (start 2.3 1.5) (end -2.3 1.5) (layer B.Fab) (width 0.1))
+    (fp_line (start -3.5 1.75) (end 3.5 1.75) (layer B.CrtYd) (width 0.05))
+    (fp_line (start 3.5 1.75) (end 3.5 -1.75) (layer B.CrtYd) (width 0.05))
+    (fp_line (start 3.5 -1.75) (end -3.5 -1.75) (layer B.CrtYd) (width 0.05))
+    (fp_line (start -3.5 -1.75) (end -3.5 1.75) (layer B.CrtYd) (width 0.05))
+    (fp_line (start -0.64944 -0.00102) (end -1.55114 -0.00102) (layer B.Fab) (width 0.1))
+    (fp_line (start 0.50118 -0.00102) (end 1.4994 -0.00102) (layer B.Fab) (width 0.1))
+    (fp_line (start -0.64944 0.79908) (end -0.64944 -0.80112) (layer B.Fab) (width 0.1))
+    (fp_line (start 0.50118 -0.75032) (end 0.50118 0.79908) (layer B.Fab) (width 0.1))
+    (fp_line (start -0.64944 -0.00102) (end 0.50118 -0.75032) (layer B.Fab) (width 0.1))
+    (fp_line (start -0.64944 -0.00102) (end 0.50118 0.79908) (layer B.Fab) (width 0.1))
+    (fp_line (start -3.4 -1.65) (end 2 -1.65) (layer B.SilkS) (width 0.12))
+    (fp_line (start -3.4 1.65) (end 2 1.65) (layer B.SilkS) (width 0.12))
+    (pad 1 smd rect (at -2 0 180) (size 2.5 1.8) (layers B.Cu B.Paste B.Mask)
+      (net 211 /SEQUENCER/VDD_IN))
+    (pad 2 smd rect (at 2 0 180) (size 2.5 1.8) (layers B.Cu B.Paste B.Mask)
+      (net 213 /SEQUENCER/INA_GND))
+    (model ${KISYS3DMOD}/Diode_SMD.3dshapes/D_SMA.wrl
+      (at (xyz 0 0 0))
+      (scale (xyz 1 1 1))
+      (rotate (xyz 0 0 0))
+    )
+  )
   (dimension 24 (width 0.15) (layer Dwgs.User)
     (gr_text "24.000 mm" (at 251.3 62 90) (layer Dwgs.User)
@@
   (segment (start 167 95.8) (end 168.4 95.8) (width 0.5) (layer F.Cu) (net 1))
   (segment (start 165.9 101.45) (end 165.9 96.9) (width 0.5) (layer F.Cu) (net 1))
+  (segment (start 119.625 107.85) (end 119.575 107.8) (width 0.5) (layer F.Cu) (net 1))
+  (segment (start 119.625 110.2) (end 119.625 107.85) (width 0.5) (layer F.Cu) (net 1))
   (segment (start 48 56.45) (end 48.05 56.5) (width 0.5) (layer F.Cu) (net 2))
   (segment (start 48 54) (end 48 56.45) (width 0.5) (layer F.Cu) (net 2))
@@
   (segment (start 223.91 118.115) (end 224 118.025) (width 0.5) (layer B.Cu) (net 211))
   (segment (start 223.91 123.29) (end 223.91 118.115) (width 0.5) (layer B.Cu) (net 211))
-  (segment (start 219.825 111.475) (end 219.9 111.4) (width 0.5) (layer B.Cu) (net 211))
-  (segment (start 219.825 114.1) (end 219.825 111.475) (width 0.5) (layer B.Cu) (net 211))
   (via (at 205 125) (size 1.44) (drill 0.8) (layers F.Cu B.Cu) (net 211))
   (via (at 208 125) (size 1.44) (drill 0.8) (layers F.Cu B.Cu) (net 211))
@@
   (via (at 215.5 128) (size 1.44) (drill 0.8) (layers F.Cu B.Cu) (net 211))
   (via (at 218.5 128) (size 1.44) (drill 0.8) (layers F.Cu B.Cu) (net 211))
+  (segment (start 219.825 112.325) (end 218.75 111.25) (width 0.5) (layer B.Cu) (net 211))
+  (segment (start 219.825 114.1) (end 219.825 112.325) (width 0.5) (layer B.Cu) (net 211))
   (via (at 212.5 83) (size 1.44) (drill 0.8) (layers F.Cu B.Cu) (net 212))
   (via (at 218.5 83) (size 1.44) (drill 0.8) (layers F.Cu B.Cu) (net 212))
@@
   (segment (start 217.775 115.825) (end 218 116.05) (width 0.5) (layer B.Cu) (net 213))
   (segment (start 217.775 114.1) (end 217.775 115.825) (width 0.5) (layer B.Cu) (net 213))
-  (segment (start 214.1 112.4) (end 215.1 111.4) (width 0.5) (layer B.Cu) (net 213))
-  (segment (start 214.1 113.975) (end 214.1 112.4) (width 0.5) (layer B.Cu) (net 213))
   (segment (start 217.65 113.975) (end 217.775 114.1) (width 0.5) (layer B.Cu) (net 213))
   (segment (start 214.1 113.975) (end 217.65 113.975) (width 0.5) (layer B.Cu) (net 213))
+  (segment (start 214.1 111.9) (end 214.75 111.25) (width 0.5) (layer B.Cu) (net 213))
+  (segment (start 214.1 113.975) (end 214.1 111.9) (width 0.5) (layer B.Cu) (net 213))
   (segment (start 132.925 134.4) (end 132.925 136.4) (width 0.5) (layer F.Cu) (net 214))
   (segment (start 133.6 136.4) (end 132.925 136.4) (width 0.5) (layer F.Cu) (net 214))
