File: INTERLOCK.sch (KiCad schematic (older format))
At the start: 161 parts, among them Q301 BC857, Q302 BC857, Q303 BC857, Q304 BC857, Q305 BC857, Q306 BC857, Q307 BC857, Q308 BC857, Q309 BC857, Q310 BC857, Q311 BC857, Q312 BC857, Q313 DTC124E, Q314 DTC124E, Q315 DTC124E, Q316 DTC124E, Q317 BC857, Q318 BC857, Q319 BC857, Q320 BC857, Q321 DTA124E, Q322 DTA124E, Q323 BC857, Q324 BC857, Q325 DTC124E, Q326 DTC124E, Q327 DTC124E, Q328 DTC124E, Q329 DTC124E, Q330 DTC124E, Q331 DTC124E, Q332 DTA124E, SW301 RESET, U301 LM339, U302 MC33079, U303 MC33079, U304 LM339

Commit message: Review 1
Connections:
- net ILK_CMD renamed ILK_CMD_PI
Changed lines of the file:
@@
 Sheet 3 4
 Title "RF Amplifier Controller"
-Date "2019-11-23"
+Date "2019-12-01"
 Rev "1"
 Comp "HB9GKW"
@@
 	14175 8300 14175 7925
 Text GLabel 13775 8500 0    50   Input ~ 0
-ILK_CMD
+ILK_CMD_PI
 Wire Wire Line
 	13775 8500 13825 8500

Commit message: Review
Parts:
- D305, D306, D307, D308, D314, D315, D316, D317, D319: value DZ2S047X0L -> BZT52C4V7T-7
Changed lines of the file:
@@
 Sheet 3 4
 Title "RF Amplifier Controller"
-Date "2019-12-01"
+Date "2020-01-19"
 Rev "1"
 Comp "HB9GKW"
@@
 P 4425 2400
 F 0 "D305" H 4350 2500 50  0000 L CNN
-F 1 "DZ2S047X0L" H 4100 2300 50  0000 L CNN
+F 1 "BZT52C4V7T-7" H 4100 2300 50  0000 L CNN
 F 2 "Diode_SMD:D_SOD-523" H 4425 2225 50  0001 C CNN
-F 3 "https://industrial.panasonic.com/content/data/SC/ds/ds4/DZ2S04700L_E.pdf" H 4425 2400 50  0001 C CNN
+F 3 "https://www.mouser.ch/datasheet/2/115/ds30502-1142513.pdf" H 4425 2400 50  0001 C CNN
 	1    4425 2400
 	0    1    1    0
@@
 AR Path="/5C000D65/62FE001A" Ref="R?"  Part="1"
 AR Path="/5E11E288/62FE001A" Ref="R381"  Part="1"
-F 0 "R381" V 15175 7775 50  0000 R CNN
+F 0 "R381" V 15175 7825 50  0000 R CNN
 F 1 "470" V 15100 7800 50  0000 R CNN
 F 2 "Resistor_SMD:R_0805_2012Metric_Pad1.15x1.40mm_HandSolder" V 14955 7725 50  0001 C CNN
@@
 P 15025 8175
 F 0 "D319" H 14950 8275 50  0000 L CNN
-F 1 "DZ2S047X0L" H 14700 8075 50  0000 L CNN
+F 1 "BZT52C4V7T-7" H 14700 8075 50  0000 L CNN
 F 2 "Diode_SMD:D_SOD-523" H 15025 8000 50  0001 C CNN
-F 3 "https://industrial.panasonic.com/content/data/SC/ds/ds4/DZ2S04700L_E.pdf" H 15025 8175 50  0001 C CNN
+F 3 "https://www.mouser.ch/datasheet/2/115/ds30502-1142513.pdf" H 15025 8175 50  0001 C CNN
 	1    15025 8175
 	0    1    1    0
@@
 AR Path="/5C000D65/630CD067" Ref="R?"  Part="1"
 AR Path="/5E11E288/630CD067" Ref="R380"  Part="1"
-F 0 "R380" V 14800 7775 50  0000 R CNN
+F 0 "R380" V 14800 7825 50  0000 R CNN
 F 1 "4k7" V 14725 7800 50  0000 R CNN
 F 2 "Resistor_SMD:R_0805_2012Metric_Pad1.15x1.40mm_HandSolder" V 14580 7725 50  0001 C CNN
@@
 P 4425 4700
 F 0 "D306" H 4350 4800 50  0000 L CNN
-F 1 "DZ2S047X0L" H 4100 4600 50  0000 L CNN
+F 1 "BZT52C4V7T-7" H 4100 4600 50  0000 L CNN
 F 2 "Diode_SMD:D_SOD-523" H 4425 4525 50  0001 C CNN
-F 3 "https://industrial.panasonic.com/content/data/SC/ds/ds4/DZ2S04700L_E.pdf" H 4425 4700 50  0001 C CNN
+F 3 "https://www.mouser.ch/datasheet/2/115/ds30502-1142513.pdf" H 4425 4700 50  0001 C CNN
 	1    4425 4700
 	0    1    1    0
@@
 P 4425 7000
 F 0 "D307" H 4350 7100 50  0000 L CNN
-F 1 "DZ2S047X0L" H 4100 6900 50  0000 L CNN
+F 1 "BZT52C4V7T-7" H 4100 6900 50  0000 L CNN
 F 2 "Diode_SMD:D_SOD-523" H 4425 6825 50  0001 C CNN
-F 3 "https://industrial.panasonic.com/content/data/SC/ds/ds4/DZ2S04700L_E.pdf" H 4425 7000 50  0001 C CNN
+F 3 "https://www.mouser.ch/datasheet/2/115/ds30502-1142513.pdf" H 4425 7000 50  0001 C CNN
 	1    4425 7000
 	0    1    1    0
@@
 P 4425 9300
 F 0 "D308" H 4350 9400 50  0000 L CNN
-F 1 "DZ2S047X0L" H 4100 9200 50  0000 L CNN
+F 1 "BZT52C4V7T-7" H 4100 9200 50  0000 L CNN
 F 2 "Diode_SMD:D_SOD-523" H 4425 9125 50  0001 C CNN
-F 3 "https://industrial.panasonic.com/content/data/SC/ds/ds4/DZ2S04700L_E.pdf" H 4425 9300 50  0001 C CNN
+F 3 "https://www.mouser.ch/datasheet/2/115/ds30502-1142513.pdf" H 4425 9300 50  0001 C CNN
 	1    4425 9300
 	0    1    1    0
@@
 P 8100 2400
 F 0 "D314" H 8025 2500 50  0000 L CNN
-F 1 "DZ2S047X0L" H 7775 2300 50  0000 L CNN
+F 1 "BZT52C4V7T-7" H 7775 2300 50  0000 L CNN
 F 2 "Diode_SMD:D_SOD-523" H 8100 2225 50  0001 C CNN
-F 3 "https://industrial.panasonic.com/content/data/SC/ds/ds4/DZ2S04700L_E.pdf" H 8100 2400 50  0001 C CNN
+F 3 "https://www.mouser.ch/datasheet/2/115/ds30502-1142513.pdf" H 8100 2400 50  0001 C CNN
 	1    8100 2400
 	0    1    1    0
@@
 P 8100 6825
 F 0 "D315" H 8025 6925 50  0000 L CNN
-F 1 "DZ2S047X0L" H 7775 6725 50  0000 L CNN
+F 1 "BZT52C4V7T-7" H 7775 6725 50  0000 L CNN
 F 2 "Diode_SMD:D_SOD-523" H 8100 6650 50  0001 C CNN
-F 3 "https://industrial.panasonic.com/content/data/SC/ds/ds4/DZ2S04700L_E.pdf" H 8100 6825 50  0001 C CNN
+F 3 "https://www.mouser.ch/datasheet/2/115/ds30502-1142513.pdf" H 8100 6825 50  0001 C CNN
 	1    8100 6825
 	0    1    1    0
@@
 P 8100 9125
 F 0 "D316" H 8025 9225 50  0000 L CNN
-F 1 "DZ2S047X0L" H 7775 9025 50  0000 L CNN
+F 1 "BZT52C4V7T-7" H 7775 9025 50  0000 L CNN
 F 2 "Diode_SMD:D_SOD-523" H 8100 8950 50  0001 C CNN
-F 3 "https://industrial.panasonic.com/content/data/SC/ds/ds4/DZ2S04700L_E.pdf" H 8100 9125 50  0001 C CNN
+F 3 "https://www.mouser.ch/datasheet/2/115/ds30502-1142513.pdf" H 8100 9125 50  0001 C CNN
 	1    8100 9125
 	0    1    1    0
@@
 P 8125 4700
 F 0 "D317" H 8050 4800 50  0000 L CNN
-F 1 "DZ2S047X0L" H 7800 4600 50  0000 L CNN
+F 1 "BZT52C4V7T-7" H 7800 4600 50  0000 L CNN
 F 2 "Diode_SMD:D_SOD-523" H 8125 4525 50  0001 C CNN
-F 3 "https://industrial.panasonic.com/content/data/SC/ds/ds4/DZ2S04700L_E.pdf" H 8125 4700 50  0001 C CNN
+F 3 "https://www.mouser.ch/datasheet/2/115/ds30502-1142513.pdf" H 8125 4700 50  0001 C CNN
 	1    8125 4700
 	0    1    1    0

Commit message: new Version with AVR Controller
Parts:
- removed C302, C303, C304, C305, C306, C307, C308, C309, C314, C315: 47n, Capacitor_SMD:C_0805_2012Metric_Pad1.15x1.40mm_HandSolder, symbol Device:C
- removed D301: HSWR1, LED_THT:LED_D3.0mm, symbol Device:LED
- removed D302: HSWR2, LED_THT:LED_D3.0mm, symbol Device:LED
- removed D303: HSWR3, LED_THT:LED_D3.0mm, symbol Device:LED
- removed D304: HSWR4, LED_THT:LED_D3.0mm, symbol Device:LED
- removed D305, D306, D307, D308, D314, D315, D316, D317, D319: BZT52C4V7T-7, Diode_SMD:D_SOD-523, symbol Diode:DZ2S047X0L
- removed D310: RF_OL, LED_THT:LED_D3.0mm, symbol Device:LED
- removed D311: TEMP1, LED_THT:LED_D3.0mm, symbol Device:LED
- removed D312: TEMP2, LED_THT:LED_D3.0mm, symbol Device:LED
- removed D313: OC, LED_THT:LED_D3.0mm, symbol Device:LED
- removed D318: FAULT, LED_THT:LED_D3.0mm, symbol Device:LED
- removed Q301, Q302, Q303, Q304, Q305, Q306, Q307, Q308, Q309, Q310, Q311, Q312, Q317, Q318, Q319, Q320, Q323, Q324: BC857, Package_TO_SOT_SMD:SOT-23, symbol Transistor_BJT:BC857
- removed Q313, Q314, Q315, Q316, Q325, Q326, Q327, Q328, Q329, Q330, Q331: DTC124E, Package_TO_SOT_SMD:SOT-23, symbol Transistor_BJT:DTC124E
- removed Q321, Q322, Q332: DTA124E, Package_TO_SOT_SMD:SOT-23, symbol Transistor_BJT:DTA124E
- removed R301, R302, R303, R304, R305, R306, R307, R308, R356, R359, R361, R362: 100k, Resistor_SMD:R_0805_2012Metric_Pad1.15x1.40mm_HandSolder, symbol Device:R
- removed R309, R310, R311, R312: 15k, Resistor_SMD:R_0805_2012Metric_Pad1.15x1.40mm_HandSolder, symbol Device:R
- removed R313, R314, R315, R316: 82k, Resistor_SMD:R_0805_2012Metric_Pad1.15x1.40mm_HandSolder, symbol Device:R
- removed R317, R318, R319, R320, R354, R357, R379: 47k, Resistor_SMD:R_0805_2012Metric_Pad1.15x1.40mm_HandSolder, symbol Device:R
- removed R321, R322, R323, R324, R337, R339, R341, R343, R355, R358, R367, R371: 10k, Resistor_SMD:R_0805_2012Metric_Pad1.15x1.40mm_HandSolder, symbol Device:R
- removed R325, R326, R327, R328, R333, R334, R335, R336, R363, R364, R365, R366, R378: 22k, Resistor_SMD:R_0805_2012Metric_Pad1.15x1.40mm_HandSolder, symbol Device:R
- removed R329, R330, R331, R332: 820k, Resistor_SMD:R_0805_2012Metric_Pad1.15x1.40mm_HandSolder, symbol Device:R
- removed R338, R340, R342, R344, R368, R369, R370, R372, R380: 4k7, Resistor_SMD:R_0805_2012Metric_Pad1.15x1.40mm_HandSolder, symbol Device:R
- removed R345, R346, R347, R348, R373, R374, R375, R376, R381: 470, Resistor_SMD:R_0805_2012Metric_Pad1.15x1.40mm_HandSolder, symbol Device:R
- removed R377: 1k, Resistor_SMD:R_0805_2012Metric_Pad1.15x1.40mm_HandSolder, symbol Device:R
- removed RV301, RV302, RV303, RV304, RV307, RV308: 50k, Potentiometer_THT:Potentiometer_Bourns_3296W_Vertical, symbol Device:R_POT_TRIM
- removed SW301: RESET, Button_Switch_THT:SW_PUSH_6mm, symbol Switch:SW_Push
- removed unit 1 of U301
- removed unit 4 of U301
- removed unit 3 of U301
- removed unit 2 of U301
- removed unit 2 of U302
- removed unit 1 of U302
- removed unit 4 of U302
- removed unit 3 of U302
- removed unit 3 of U303
- removed unit 4 of U303
- removed unit 2 of U303
- removed unit 1 of U303
- removed unit 4 of U304
- removed unit 2 of U304
- added C? (x16): 47n, Capacitor_SMD:C_0805_2012Metric_Pad1.15x1.40mm_HandSolder, symbol Device:C
- added C? (x12): 100n, Capacitor_SMD:C_0805_2012Metric_Pad1.15x1.40mm_HandSolder, symbol Device:C
- added C? (x2): 470u, Capacitor_THT:CP_Radial_D22.0mm_P10.00mm_SnapIn, symbol Device:CP
- added C? (x2): 100n, Capacitor_SMD:C_1206_3216Metric_Pad1.42x1.75mm_HandSolder, symbol Device:C
- added C? (x2): 4u7, Capacitor_Tantalum_SMD:CP_EIA-6032-28_Kemet-C, symbol Device:CP
- added D?: Z1SMA33, Diode_SMD:D_SMA, symbol Diode:Z1SMAxxx
- added D? (x2): BZT52C4V7T-7, Diode_SMD:D_SOD-523, symbol Diode:DZ2S047X0L
- added D? (x4): PMEG6010CEH, Diode_SMD:D_SOD-123, symbol Diode:PMEG6010CEH
- added FB? (x8): Ferrite_Bead_Small, Resistor_SMD:R_0805_2012Metric_Pad1.15x1.40mm_HandSolder, symbol Device:Ferrite_Bead_Small
- added Q? (x2): IXTH140P10T, Package_TO_SOT_THT:TO-247-3_Vertical, symbol Transistor_FET:SUD50P08-25L
- added Q?: BC857, Package_TO_SOT_SMD:SOT-23, symbol Transistor_BJT:BC857
- added Q? (x4): DTC124E, Package_TO_SOT_SMD:SOT-23, symbol Transistor_BJT:DTC124E
- added Q?: DTA124E, Package_TO_SOT_SMD:SOT-23, symbol Transistor_BJT:DTA124E
- added Q? (x2): BCX53, Package_TO_SOT_SMD:SOT-89-3, symbol Transistor_BJT:BCX53
- added Q? (x4): BCX56, Package_TO_SOT_SMD:SOT-89-3, symbol Transistor_BJT:BCX56
- added Q? (x2): BC847, Package_TO_SOT_SMD:SOT-23, symbol Transistor_BJT:BC847
- added R? (x4): 8k2, Resistor_SMD:R_0805_2012Metric_Pad1.15x1.40mm_HandSolder, symbol Device:R
- added R? (x10): 100k, Resistor_SMD:R_0805_2012Metric_Pad1.15x1.40mm_HandSolder, symbol Device:R
- added R? (x4): 15k, Resistor_SMD:R_0805_2012Metric_Pad1.15x1.40mm_HandSolder, symbol Device:R
- added R? (x7): 4k7, Resistor_SMD:R_0805_2012Metric_Pad1.15x1.40mm_HandSolder, symbol Device:R
- added R? (x13): 10k, Resistor_SMD:R_0805_2012Metric_Pad1.15x1.40mm_HandSolder, symbol Device:R
- added R? (x10): 1k, Resistor_SMD:R_0805_2012Metric_Pad1.15x1.40mm_HandSolder, symbol Device:R
- added R? (x6): 47k, Resistor_SMD:R_0805_2012Metric_Pad1.15x1.40mm_HandSolder, symbol Device:R
- added R? (x8): 330, Resistor_SMD:R_0805_2012Metric_Pad1.15x1.40mm_HandSolder, symbol Device:R
- added R? (x4): 0R015, Resistor_SMD:R_Shunt_Vishay_WSR2_WSR3_KelvinConnection, symbol Device:R
- added R?: 68k, Resistor_SMD:R_0805_2012Metric_Pad1.15x1.40mm_HandSolder, symbol Device:R
- added R?: 6k8, Resistor_SMD:R_0805_2012Metric_Pad1.15x1.40mm_HandSolder, symbol Device:R
- added RV? (x5): 20k, Potentiometer_THT:Potentiometer_Bourns_3296W_Vertical, symbol Device:R_POT_TRIM
- added U? (x8): MC33079, Package_SO:SOIC-14_3.9x8.7mm_P1.27mm, symbol Amplifier_Operational:MC33079
- added U? (x4): LM339, Package_SO:SOIC-14_3.9x8.7mm_P1.27mm, symbol Comparator:LM339
- added U?: INA138, Package_TO_SOT_SMD:SOT-23-5, symbol Amplifier_Current:INA138
- added U? (x6): MC33078, Package_SO:SOIC-8_3.9x4.9mm_P1.27mm, symbol Amplifier_Operational:MC33078
Connections:
- net labels added: +5V, ALC, GATE_ALC_EN, ILK_IDD_OL, RF_SW1, RF_SW1_EN, RF_SW1_ON, RF_SW1_ON_, RF_SW2, RF_SW2_EN, RF_SW2_ON, RF_SW2_ON_, VDD_EN, VDD_IN, VDD_MON, VDD_OUT, VSS_IN, VSS_OUT
- net labels removed: FAULT, FWD2_MON, FWD3, FWD3_MON, FWD4, ILK, ILK_CMD_PI, ILK_HSWR2, ILK_HSWR3, ILK_HSWR4, ILK_IDD_OC, ILK_TEMP1, ILK_TEMP2, OP, REF2_MON, REF3, REF3_MON, REF4, REF4_MON, RESET, RESET_CMD, RF_READY, TEMP1, TEMP1_MON, TEMP2, TEMP2_MON
- wire segments 463 -> 459
Other:
- moved on the sheet: C301, C310, C311, C312, C313, C316, D309, R349, R350, R351, R352, R353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
