File: SEQUENCER.sch (KiCad schematic (older format))
At the start: 118 parts, among them Q401 IXTH140P10T, Q402 IXTH140P10T, Q403 DTC124E, Q404 BC857, Q405 DTC124E, Q406 DTC124E, Q407 DTC124E, Q408 DTA124E, Q409 DTC124E, Q410 DTC124E, Q411 DTA124E, Q412 BCX53, Q413 DTA124E, Q414 DTC124E, Q415 DTC124E, Q416 BCX53, Q417 DTA124E, Q418 DTC124E, Q419 DTC124E, Q420 BCX53, Q421 DTA124E, Q422 DTC124E, Q423 DTC124E, Q424 DTC124E, Q425 DTA124E, Q426 BCX53, Q427 DTC124E, Q428 DTC124E, Q429 DTC124E, U401 MC33078, U402 MC33079, U403 INA138, U404 LM339

Commit message: Review 1
Parts:
- D401: value SMZ24 -> SMZ33
- R407: value 1k8 -> 39k
Other:
- moved on the sheet: R401, R405
Changed lines of the file:
@@
 Sheet 4 4
 Title "RF Amplifier Controller"
-Date "2019-11-23"
+Date "2019-12-01"
 Rev "1"
 Comp "HB9GKW"
@@
 	4000 2825 3875 2825
 Wire Wire Line
-	3575 2825 3575 2875
-Wire Wire Line
-	3575 3175 3575 3225
-Wire Wire Line
-	3575 3225 3875 3225
+	3500 2825 3500 2875
+Wire Wire Line
+	3500 3175 3500 3225
+Wire Wire Line
+	3500 3225 3875 3225
 Wire Wire Line
 	4000 3225 4000 3125
@@
 AR Path="/5C000D65/5D2C55AC" Ref="R?"  Part="1"
 AR Path="/5D2BEC5D/5D2C55AC" Ref="R402"  Part="1"
-F 0 "R402" H 3400 3075 50  0000 R CNN
-F 1 "0R015" H 3500 2975 50  0000 R CNN
+F 0 "R402" V 3350 3125 50  0000 R CNN
+F 1 "0R015" V 3275 3150 50  0000 R CNN
 F 2 "Resistor_SMD:R_Shunt_Vishay_WSR2_WSR3_KelvinConnection" V 3130 3025 50  0001 C CNN
 F 3 "~" H 3200 3025 50  0001 C CNN
@@
 L Device:R R?
 U 1 1 5D2C55B3
-P 2825 3025
+P 2900 3025
 AR Path="/5D2C55B3" Ref="R?"  Part="1"
 AR Path="/5C000D65/5D2C55B3" Ref="R?"  Part="1"
 AR Path="/5D2BEC5D/5D2C55B3" Ref="R401"  Part="1"
-F 0 "R401" H 3025 3075 50  0000 R CNN
-F 1 "0R015" H 3125 2975 50  0000 R CNN
-F 2 "Resistor_SMD:R_Shunt_Vishay_WSR2_WSR3_KelvinConnection" V 2755 3025 50  0001 C CNN
-F 3 "~" H 2825 3025 50  0001 C CNN
-	1    2825 3025
-	-1   0    0    -1
-$EndComp
-Wire Wire Line
-	2825 3175 2825 3225
+F 0 "R401" V 3050 3125 50  0000 R CNN
+F 1 "0R015" V 2975 3150 50  0000 R CNN
+F 2 "Resistor_SMD:R_Shunt_Vishay_WSR2_WSR3_KelvinConnection" V 2830 3025 50  0001 C CNN
+F 3 "~" H 2900 3025 50  0001 C CNN
+	1    2900 3025
+	-1   0    0    -1
+$EndComp
+Wire Wire Line
+	2900 3175 2900 3225
 Wire Wire Line
 	3200 3175 3200 3225
-Connection ~ 3575 3225
-Wire Wire Line
-	2825 2875 2825 2825
-Wire Wire Line
-	2825 2825 3200 2825
-Wire Wire Line
-	3200 2825 3575 2825
+Connection ~ 3500 3225
+Wire Wire Line
+	2900 2875 2900 2825
+Wire Wire Line
+	2900 2825 3200 2825
+Wire Wire Line
+	3200 2825 3500 2825
 Connection ~ 3200 2825
-Connection ~ 3575 2825
+Connection ~ 3500 2825
 Wire Wire Line
 	3200 2825 3200 2875
@@
 U 1 1 5D2C55D9
 P 3875 3025
-F 0 "C410" H 3725 3100 50  0000 L CNN
+F 0 "C410" H 3675 3100 50  0000 L CNN
 F 1 "100n" H 3675 2925 50  0000 L CNN
 F 2 "Capacitor_SMD:C_0805_2012Metric_Pad1.15x1.40mm_HandSolder" H 3913 2875 50  0001 C CNN
@@
 Connection ~ 3875 2825
 Wire Wire Line
-	3875 2825 3575 2825
+	3875 2825 3500 2825
 Wire Wire Line
 	3875 3175 3875 3225
@@
 	3875 3225 4000 3225
 Wire Wire Line
-	3575 3225 3200 3225
+	3500 3225 3200 3225
 Connection ~ 3200 3225
 Wire Wire Line
-	3200 3225 2825 3225
+	3200 3225 2900 3225
 $Comp
 L Amplifier_Current:INA138 U403
@@
 P 3625 2000
 F 0 "D401" H 3625 2216 50  0000 C CNN
-F 1 "SMZ24" H 3625 2125 50  0000 C CNN
+F 1 "SMZ33" H 3625 2125 50  0000 C CNN
 F 2 "Diode_SMD:D_MELF" H 3625 1825 50  0001 C CNN
 F 3 "https://diotec.com/tl_files/diotec/files/pdf/datasheets/smz1.pdf" H 3625 2000 50  0001 C CNN
@@
 AR Path="/5C000D65/5D2C5613" Ref="R?"  Part="1"
 AR Path="/5D2BEC5D/5D2C5613" Ref="R407"  Part="1"
-F 0 "R407" H 3755 2296 50  0000 R CNN
-F 1 "1k8" H 3755 2205 50  0000 R CNN
+F 0 "R407" V 3975 2350 50  0000 R CNN
+F 1 "39k" V 3900 2325 50  0000 R CNN
 F 2 "Resistor_SMD:R_0805_2012Metric_Pad1.15x1.40mm_HandSolder" V 3755 2250 50  0001 C CNN
 F 3 "~" H 3825 2250 50  0001 C CNN
@@
 U 1 1 5D2C5628
 P 4400 2250
-F 0 "C411" H 4250 2350 50  0000 L CNN
-F 1 "100n" H 4200 2150 50  0000 L CNN
+F 0 "C411" H 4425 2350 50  0000 L CNN
+F 1 "100n" H 4450 2150 50  0000 L CNN
 F 2 "Capacitor_SMD:C_0805_2012Metric_Pad1.15x1.40mm_HandSolder" H 4438 2100 50  0001 C CNN
 F 3 "~" H 4400 2250 50  0001 C CNN
@@
 AR Path="/5C000D65/5D2C5646" Ref="R?"  Part="1"
 AR Path="/5D2BEC5D/5D2C5646" Ref="R409"  Part="1"
-F 0 "R409" H 5355 3646 50  0000 R CNN
-F 1 "100k" H 5355 3555 50  0000 R CNN
+F 0 "R409" V 5575 3700 50  0000 R CNN
+F 1 "100k" V 5500 3700 50  0000 R CNN
 F 2 "Resistor_SMD:R_0805_2012Metric_Pad1.15x1.40mm_HandSolder" V 5355 3600 50  0001 C CNN
 F 3 "~" H 5425 3600 50  0001 C CNN
@@
 AR Path="/5C000D65/5D2C5698" Ref="R?"  Part="1"
 AR Path="/5D2BEC5D/5D2C5698" Ref="R404"  Part="1"
-F 0 "R404" V 3375 4200 50  0000 R CNN
-F 1 "10k" V 3300 4175 50  0000 R CNN
+F 0 "R404" V 3625 4200 50  0000 R CNN
+F 1 "10k" V 3550 4175 50  0000 R CNN
 F 2 "Resistor_SMD:R_0805_2012Metric_Pad1.15x1.40mm_HandSolder" V 3405 4100 50  0001 C CNN
 F 3 "~" H 3475 4100 50  0001 C CNN
@@
 AR Path="/5C000D65/5D2C56A3" Ref="R?"  Part="1"
 AR Path="/5D2BEC5D/5D2C56A3" Ref="R408"  Part="1"
-F 0 "R408" V 3825 4450 50  0000 R CNN
-F 1 "68k" V 3750 4425 50  0000 R CNN
+F 0 "R408" V 4075 4450 50  0000 R CNN
+F 1 "68k" V 4000 4425 50  0000 R CNN
 F 2 "Resistor_SMD:R_0805_2012Metric_Pad1.15x1.40mm_HandSolder" V 3855 4350 50  0001 C CNN
 F 3 "~" H 3925 4350 50  0001 C CNN
@@
 AR Path="/5C000D65/5D8DD977" Ref="R?"  Part="1"
 AR Path="/5D2BEC5D/5D8DD977" Ref="R406"  Part="1"
-F 0 "R406" H 3630 5946 50  0000 R CNN
-F 1 "10k" H 3630 5855 50  0000 R CNN
+F 0 "R406" V 3875 6000 50  0000 R CNN
+F 1 "10k" V 3800 5975 50  0000 R CNN
 F 2 "Resistor_SMD:R_0805_2012Metric_Pad1.15x1.40mm_HandSolder" V 3630 5900 50  0001 C CNN
 F 3 "~" H 3700 5900 50  0001 C CNN
@@
 AR Path="/5C000D65/5D8DD988" Ref="R?"  Part="1"
 AR Path="/5D2BEC5D/5D8DD988" Ref="R403"  Part="1"
-F 0 "R403" V 3350 5675 50  0000 R CNN
-F 1 "100k" V 3275 5725 50  0000 R CNN
+F 0 "R403" V 3600 5750 50  0000 R CNN
+F 1 "100k" V 3525 5750 50  0000 R CNN
 F 2 "Resistor_SMD:R_0805_2012Metric_Pad1.15x1.40mm_HandSolder" V 3380 5650 50  0001 C CNN
 F 3 "~" H 3450 5650 50  0001 C CNN
@@
 AR Path="/5D8DD992" Ref="C?"  Part="1"
 AR Path="/5D2BEC5D/5D8DD992" Ref="C404"  Part="1"
-F 0 "C404" H 2575 5950 50  0000 L CNN
-F 1 "470u" H 2575 5800 50  0000 L CNN
+F 0 "C404" H 2525 6000 50  0000 L CNN
+F 1 "470u" H 2550 5800 50  0000 L CNN
 F 2 "Capacitor_THT:CP_Radial_D22.0mm_P10.00mm_SnapIn" H 2863 5750 50  0001 C CNN
 F 3 "~" H 2825 5900 50  0001 C CNN
@@
 AR Path="/5D8DD9A4" Ref="C?"  Part="1"
 AR Path="/5D2BEC5D/5D8DD9A4" Ref="C407"  Part="1"
-F 0 "C407" H 2975 5950 50  0000 L CNN
+F 0 "C407" H 2975 6000 50  0000 L CNN
 F 1 "100n" H 2975 5800 50  0000 L CNN
 F 2 "Capacitor_SMD:C_0805_2012Metric_Pad1.15x1.40mm_HandSolder" H 3238 5750 50  0001 C CNN
@@
 AR Path="/5D3509AC" Ref="C?"  Part="1"
 AR Path="/5D2BEC5D/5D3509AC" Ref="C409"  Part="1"
-F 0 "C409" H 3450 5175 50  0000 L CNN
-F 1 "100n" H 3450 5025 50  0000 L CNN
+F 0 "C409" H 3725 5225 50  0000 L CNN
+F 1 "100n" H 3750 5025 50  0000 L CNN
 F 2 "Capacitor_SMD:C_0805_2012Metric_Pad1.15x1.40mm_HandSolder" H 3713 4975 50  0001 C CNN
 F 3 "~" H 3675 5125 50  0001 C CNN
@@
 L Device:R R?
 U 1 1 5D2C559D
-P 3575 3025
+P 3500 3025
 AR Path="/5D2C559D" Ref="R?"  Part="1"
 AR Path="/5C000D65/5D2C559D" Ref="R?"  Part="1"
 AR Path="/5D2BEC5D/5D2C559D" Ref="R405"  Part="1"
-F 0 "R405" H 3775 3075 50  0000 R CNN
-F 1 "0R015" H 3875 2975 50  0000 R CNN
-F 2 "Resistor_SMD:R_Shunt_Vishay_WSR2_WSR3_KelvinConnection" V 3505 3025 50  0001 C CNN
-F 3 "~" H 3575 3025 50  0001 C CNN
-	1    3575 3025
-	-1   0    0    -1
-$EndComp
+F 0 "R405" V 3650 3125 50  0000 R CNN
+F 1 "0R015" V 3575 3150 50  0000 R CNN
+F 2 "Resistor_SMD:R_Shunt_Vishay_WSR2_WSR3_KelvinConnection" V 3430 3025 50  0001 C CNN
+F 3 "~" H 3500 3025 50  0001 C CNN
+	1    3500 3025
+	-1   0    0    -1
+$EndComp

Commit message: Review 2
Parts:
- removed D401: SMZ33, Diode_SMD:D_MELF, symbol Diode:SMZxxx
- added D401: Z1SMA33, Diode_SMD:D_SMA, symbol Diode:Z1SMAxxx
- R406: value 10k -> 6k8
- R407: value 39k -> 4k7
Changed lines of the file:
@@
 EESchema Schematic File Version 4
-LIBS:RF-AMP-CNTLR_V1-cache
 EELAYER 30 0
 EELAYER END
@@
 Sheet 4 4
 Title "RF Amplifier Controller"
-Date "2019-12-01"
+Date "2020-01-11"
 Rev "1"
 Comp "HB9GKW"
@@
 $EndComp
 $Comp
-L Diode:SMZxxx D401
-U 1 1 5D2C560C
-P 3625 2000
-F 0 "D401" H 3625 2216 50  0000 C CNN
-F 1 "SMZ33" H 3625 2125 50  0000 C CNN
-F 2 "Diode_SMD:D_MELF" H 3625 1825 50  0001 C CNN
-F 3 "https://diotec.com/tl_files/diotec/files/pdf/datasheets/smz1.pdf" H 3625 2000 50  0001 C CNN
-	1    3625 2000
-	1    0    0    -1
-$EndComp
-$Comp
 L Device:R R?
 U 1 1 5D2C5613
@@
 AR Path="/5D2BEC5D/5D2C5613" Ref="R407"  Part="1"
 F 0 "R407" V 3975 2350 50  0000 R CNN
-F 1 "39k" V 3900 2325 50  0000 R CNN
+F 1 "4k7" V 3900 2325 50  0000 R CNN
 F 2 "Resistor_SMD:R_0805_2012Metric_Pad1.15x1.40mm_HandSolder" V 3755 2250 50  0001 C CNN
 F 3 "~" H 3825 2250 50  0001 C CNN
@@
 AR Path="/5D2BEC5D/5D8DD977" Ref="R406"  Part="1"
 F 0 "R406" V 3875 6000 50  0000 R CNN
-F 1 "10k" V 3800 5975 50  0000 R CNN
+F 1 "6k8" V 3800 5975 50  0000 R CNN
 F 2 "Resistor_SMD:R_0805_2012Metric_Pad1.15x1.40mm_HandSolder" V 3630 5900 50  0001 C CNN
 F 3 "~" H 3700 5900 50  0001 C CNN
@@
 Wire Notes Line
 	1900 825  7025 825
+$Comp
+L Diode:Z1SMAxxx D401
+U 1 1 5E1D16AF
+P 3625 2000
+F 0 "D401" H 3625 2216 50  0000 C CNN
+F 1 "Z1SMA33" H 3625 2125 50  0000 C CNN
+F 2 "Diode_SMD:D_SMA" H 3625 1825 50  0001 C CNN
+F 3 "https://diotec.com/tl_files/diotec/files/pdf/datasheets/z1sma1.pdf" H 3625 2000 50  0001 C CNN
+	1    3625 2000
+	1    0    0    -1
+$EndComp
 $EndSCHEMATC

Commit message: Review
Parts:
- D402: value DZ2S130X0L -> BZT52C13T-7
- D404, D406, D409, D410, D413, D414: value DZ2S047X0L -> BZT52C4V7T-7
- D405: value DZ2S030X0L -> BZT52C13T-7
Other:
- moved on the sheet: C404

Commit message: new Version with AVR Controller
Parts:
- removed C401, C402, C405, C406, C407, C408, C409, C410, C411, C412, C413, C414, C415, C416, C417, C418, C419, C423, C427: 100n, Capacitor_SMD:C_0805_2012Metric_Pad1.15x1.40mm_HandSolder, symbol Device:C
- removed C403, C404: 470u, Capacitor_THT:CP_Radial_D22.0mm_P10.00mm_SnapIn, symbol Device:CP
- removed C420, C421, C424, C425: 1u, Capacitor_SMD:C_0805_2012Metric_Pad1.15x1.40mm_HandSolder, symbol Device:C
- removed C422, C426: 4u7, Capacitor_Tantalum_SMD:CP_EIA-6032-28_Kemet-C, symbol Device:CP
- removed D401: Z1SMA33, Diode_SMD:D_SMA, symbol Diode:Z1SMAxxx
- removed D402: BZT52C13T-7, Diode_SMD:D_SOD-523, symbol Diode:DZ2S130X0L
- removed D403: DZ2S047X0L, Diode_SMD:D_SOD-523, symbol Diode:DZ2S047X0L
- removed D404, D406, D409, D410, D413, D414: BZT52C4V7T-7, Diode_SMD:D_SOD-523, symbol Diode:DZ2S047X0L
- removed D405: BZT52C13T-7, Diode_SMD:D_SOD-523, symbol Diode:DZ2S030X0L
- removed D407, D408, D411, D412: PMEG6010CEH, Diode_SMD:D_SOD-123, symbol Diode:PMEG6010CEH
- removed JP401, JP402: SolderJumper_2_Open, Jumper:SolderJumper-2_P1.3mm_Open_Pad1.0x1.5mm, symbol Jumper:SolderJumper_2_Open
- removed Q401, Q402: IXTH140P10T, Package_TO_SOT_THT:TO-247-3_Vertical, symbol Transistor_FET:SUD50P08-25L
- removed Q403, Q405, Q406, Q407, Q409, Q410, Q414, Q415, Q418, Q419, Q422, Q423, Q424, Q427, Q428, Q429: DTC124E, Package_TO_SOT_SMD:SOT-23, symbol Transistor_BJT:DTC124E
- removed Q404: BC857, Package_TO_SOT_SMD:SOT-23, symbol Transistor_BJT:BC857
- removed Q408, Q411, Q413, Q417, Q421, Q425: DTA124E, Package_TO_SOT_SMD:SOT-23, symbol Transistor_BJT:DTA124E
- removed Q412, Q416, Q420, Q426: BCX53, Package_TO_SOT_SMD:SOT-89-3, symbol Transistor_BJT:BCX53
- removed R401, R402, R405: 0R015, Resistor_SMD:R_Shunt_Vishay_WSR2_WSR3_KelvinConnection, symbol Device:R
- removed R403, R409, R414: 100k, Resistor_SMD:R_0805_2012Metric_Pad1.15x1.40mm_HandSolder, symbol Device:R
- removed R404, R410, R413, R419, R420, R422, R423, R427, R428, R430, R431: 10k, Resistor_SMD:R_0805_2012Metric_Pad1.15x1.40mm_HandSolder, symbol Device:R
- removed R406: 6k8, Resistor_SMD:R_0805_2012Metric_Pad1.15x1.40mm_HandSolder, symbol Device:R
- removed R407: 4k7, Resistor_SMD:R_0805_2012Metric_Pad1.15x1.40mm_HandSolder, symbol Device:R
- removed R408: 68k, Resistor_SMD:R_0805_2012Metric_Pad1.15x1.40mm_HandSolder, symbol Device:R
- removed R411, R418, R421, R426, R429: 47k, Resistor_SMD:R_0805_2012Metric_Pad1.15x1.40mm_HandSolder, symbol Device:R
- removed R412, R415, R417, R424, R425, R432, R433, R434, R435, R436, R437: 1k, Resistor_SMD:R_0805_2012Metric_Pad1.15x1.40mm_HandSolder, symbol Device:R
- removed R416: 33k, Resistor_SMD:R_0805_2012Metric_Pad1.15x1.40mm_HandSolder, symbol Device:R
- removed RV401, RV402, RV403, RV404, RV405: 20k, Potentiometer_THT:Potentiometer_Bourns_3296W_Vertical, symbol Device:R_POT_TRIM
- removed U401: MC33078, Package_SO:SOIC-8_3.9x4.9mm_P1.27mm, symbol Amplifier_Operational:MC33078
- removed U402: MC33079, Package_SO:SOIC-14_3.9x8.7mm_P1.27mm, symbol Amplifier_Operational:MC33079
- removed U403: INA138, Package_TO_SOT_SMD:SOT-23-5, symbol Amplifier_Current:INA138
- removed U404: LM339, Package_SO:SOIC-14_3.9x8.7mm_P1.27mm, symbol Comparator:LM339
Other:
- note removed: "3x WSHM2818"
