File: RF-AMP-CNTLR_V1.sch (KiCad schematic (older format))
At the start: 69 parts, among them J101 VAC, J102 VDC, J103 ext_13V8, J104 Front Panel, J105 ANT_SWITCH, J106 BAND_SELECT, J107 I2C0, J108 VDD_IN, J109 VSS_IN, J110 RELAY RF OUT, J111 RELAY RF IN, J112 FWD3, J113 REF3, J114 FWD4, J115 REF4, J116 PTT, J117 ALC, J118 VDD_AMP, J119 GND_AMP, J120 SPI0, J121 I2C1, J122 RS232, J123 AMP1, J124 AMP2, Q101 DTA124E, U101 KA378R12C, U102 SFH617A-2, U103 L78L33_SOT89

Commit message: Review 1
Parts:
- removed C105: 470n, Capacitor_THT:C_Rect_L7.0mm_W3.5mm_P5.00mm, symbol Device:C
- added C105: 47u, Capacitor_Tantalum_SMD:CP_EIA-6032-28_Kemet-C, symbol Device:CP
- added D103, D104: BAT54CW, Package_TO_SOT_SMD:SOT-323_SC-70, symbol Diode:BAT54CW
- C108: value 33n -> 470n
- R103: value 470k -> 620
Connections:
- net CONTROLLER/INT_OC is gone; now on net CONTROLLER/INT_OC: J107.4 (Pin_4)
- net CONTROLLER/INT_OC: no longer J121.4 (Pin_4)
- net OP: now also D103.3; no longer J104.16 (Pin_16)
- net RESET_CMD: now also D104.3; no longer J104.12 (Pin_12)
- net at C103.2, C109.1, FL101.4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: no longer D101.3 (~~)
- net at C108.2, D101.4 (~~): no longer C109.2
- net at D101.2 (-), U102.2: now also C105.2
- net at D101.1 (+), R103.1: now also C105.1
- new net: C109.2, D101.3 (~~)
- new net: D104.1, J104.12 (Pin_12)
- new net: D103.1, J104.16 (Pin_16)
- new net CONTROLLER/INT_OC: J121.4 (Pin_4)
- new net OP_CMD_PI: D103.2
- new net RESET_CMD_PI: D104.2
Other:
- moved on the sheet: C109, D101, R103, U102
Changed lines of the file:
@@
 Sheet 1 4
 Title "RF Amplifier Controller"
-Date "2019-11-23"
+Date "2019-12-01"
 Rev "1"
 Comp "HB9GKW"
@@
 $EndComp
 Wire Wire Line
-	5475 2150 5475 2325
-Wire Wire Line
 	5475 3150 5900 3150
 Connection ~ 5475 2150
@@
 L Device:C C?
 U 1 1 5D83FED4
-P 5250 2325
+P 5250 2825
 AR Path="/5CBB0B33/5D83FED4" Ref="C?"  Part="1"
 AR Path="/5D83FED4" Ref="C109"  Part="1"
-F 0 "C109" V 5100 2250 50  0000 L CNN
-F 1 "470n" V 5400 2250 50  0000 L CNN
-F 2 "Capacitor_THT:C_Rect_L7.0mm_W3.5mm_P5.00mm" H 5288 2175 50  0001 C CNN
-F 3 "~" H 5250 2325 50  0001 C CNN
-	1    5250 2325
+F 0 "C109" V 5100 2750 50  0000 L CNN
+F 1 "470n" V 5400 2750 50  0000 L CNN
+F 2 "Capacitor_THT:C_Rect_L7.0mm_W3.5mm_P5.00mm" H 5288 2675 50  0001 C CNN
+F 3 "~" H 5250 2825 50  0001 C CNN
+	1    5250 2825
 	0    1    1    0
 $EndComp
@@
 L Isolator:SFH617A-2 U102
 U 1 1 5D867C9D
-P 3825 3025
-F 0 "U102" H 3825 3350 50  0000 C CNN
-F 1 "SFH617A-2" H 3825 3259 50  0000 C CNN
-F 2 "Package_DIP:DIP-4_W7.62mm" H 3625 2825 50  0001 L CIN
-F 3 "http://www.vishay.com/docs/83740/sfh617a.pdf" H 3825 3025 50  0001 L CNN
-	1    3825 3025
+P 3475 3025
+F 0 "U102" H 3475 2825 50  0000 C CNN
+F 1 "SFH617A-2" H 3475 2750 50  0000 C CNN
+F 2 "Package_DIP:DIP-4_W7.62mm" H 3275 2825 50  0001 L CIN
+F 3 "http://www.vishay.com/docs/83740/sfh617a.pdf" H 3475 3025 50  0001 L CNN
+	1    3475 3025
 	-1   0    0    -1
 $EndComp
@@
 L Device:R R?
 U 1 1 5D8868B9
-P 4275 2700
+P 3875 2700
 AR Path="/5CBB0B33/5D8868B9" Ref="R?"  Part="1"
 AR Path="/5D8868B9" Ref="R103"  Part="1"
-F 0 "R103" H 4025 2775 50  0000 L CNN
-F 1 "470k" H 4025 2700 50  0000 L CNN
-F 2 "Resistor_SMD:R_0805_2012Metric_Pad1.15x1.40mm_HandSolder" V 4205 2700 50  0001 C CNN
-F 3 "~" H 4275 2700 50  0001 C CNN
-	1    4275 2700
+F 0 "R103" H 3625 2775 50  0000 L CNN
+F 1 "620" H 3625 2700 50  0000 L CNN
+F 2 "Resistor_SMD:R_0805_2012Metric_Pad1.15x1.40mm_HandSolder" V 3805 2700 50  0001 C CNN
+F 3 "~" H 3875 2700 50  0001 C CNN
+	1    3875 2700
 	1    0    0    -1
 $EndComp
@@
 L Diode_Bridge:B80C800DM D101
 U 1 1 5D88948A
-P 5025 2825
-F 0 "D101" V 5225 2625 50  0000 R CNN
-F 1 "B80C800DM" V 5150 2625 50  0000 R CNN
-F 2 "Diode_THT:Diode_Bridge_DIP-4_W7.62mm_P5.08mm" H 5175 2950 50  0001 L CNN
-F 3 "https://www.vishay.com/docs/88533/800dm.pdf" H 5025 2825 50  0001 C CNN
-	1    5025 2825
-	0    -1   -1   0
-$EndComp
-Wire Wire Line
-	4725 2825 4725 2325
-$Comp
-L Device:C C?
-U 1 1 5D8CF888
-P 4475 2825
-AR Path="/5CBB0B33/5D8CF888" Ref="C?"  Part="1"
-AR Path="/5D8CF888" Ref="C105"  Part="1"
-F 0 "C105" H 4500 2925 50  0000 L CNN
-F 1 "470n" H 4500 2725 50  0000 L CNN
-F 2 "Capacitor_THT:C_Rect_L7.0mm_W3.5mm_P5.00mm" H 4513 2675 50  0001 C CNN
-F 3 "~" H 4475 2825 50  0001 C CNN
-	1    4475 2825
-	1    0    0    -1
-$EndComp
-Wire Wire Line
-	4475 2675 4475 2525
-Wire Wire Line
-	4475 2525 5025 2525
-Wire Wire Line
-	4475 2975 4475 3125
-Wire Wire Line
-	4475 3125 5025 3125
-Wire Wire Line
-	4725 2325 5100 2325
+P 4800 2825
+F 0 "D101" V 5175 2775 50  0000 R CNN
+F 1 "B80C800DM" V 5075 2725 50  0000 R CNN
+F 2 "Diode_THT:Diode_Bridge_DIP-4_W7.62mm_P5.08mm" H 4950 2950 50  0001 L CNN
+F 3 "https://www.vishay.com/docs/88533/800dm.pdf" H 4800 2825 50  0001 C CNN
+	1    4800 2825
+	0    -1   -1   0
+$EndComp
 Wire Wire Line
 	3650 1700 5475 1700
@@
 AR Path="/5D902ABA" Ref="C108"  Part="1"
 F 0 "C108" V 5100 1875 50  0000 L CNN
-F 1 "33n" V 5400 1875 50  0000 L CNN
+F 1 "470n" V 5400 1875 50  0000 L CNN
 F 2 "Capacitor_THT:C_Rect_L7.0mm_W3.5mm_P5.00mm" H 5288 1800 50  0001 C CNN
 F 3 "~" H 5250 1950 50  0001 C CNN
@@
 $EndComp
 Wire Wire Line
-	5100 1950 4725 1950
-Wire Wire Line
-	4725 1950 4725 2325
-Connection ~ 4725 2325
-Wire Wire Line
 	2575 2275 2575 2925
 Connection ~ 2575 2925
 Wire Wire Line
-	4275 2550 4275 2525
-Wire Wire Line
-	4275 2525 4475 2525
-Connection ~ 4475 2525
-Wire Wire Line
-	4275 2850 4275 2925
-Wire Wire Line
-	4275 2925 4125 2925
-Wire Wire Line
-	4125 3125 4475 3125
-Connection ~ 4475 3125
+	3875 2550 3875 2525
+Wire Wire Line
+	3875 2850 3875 2925
+Wire Wire Line
+	3875 2925 3775 2925
 $Comp
 L Device:R R?
@@
 	2975 2375 3000 2375
 Wire Wire Line
-	2975 2925 3525 2925
+	2975 2925 3175 2925
 Connection ~ 2975 2925
 $Comp
 L power:Earth #PWR0112
 U 1 1 5D9DEA31
-P 3525 3125
+P 3175 3125
 AR Path="/5D9DEA31" Ref="#PWR0112"  Part="1"
 AR Path="/5C000D65/5D9DEA31" Ref="#PWR?"  Part="1"
 AR Path="/5CBB0B33/5D9DEA31" Ref="#PWR?"  Part="1"
-F 0 "#PWR0112" H 3525 2875 50  0001 C CNN
-F 1 "Earth" H 3525 2975 50  0001 C CNN
-F 2 "" H 3525 3125 50  0001 C CNN
-F 3 "" H 3525 3125 50  0001 C CNN
-	1    3525 3125
+F 0 "#PWR0112" H 3175 2875 50  0001 C CNN
+F 1 "Earth" H 3175 2975 50  0001 C CNN
+F 2 "" H 3175 3125 50  0001 C CNN
+F 3 "" H 3175 3125 50  0001 C CNN
+	1    3175 3125
 	1    0    0    -1
 $EndComp
@@
 	5400 1950 5675 1950
 Wire Wire Line
-	5400 2325 5475 2325
-Connection ~ 5475 2325
-Wire Wire Line
-	5475 2325 5475 2825
-Wire Wire Line
 	5675 1950 5675 2950
-Wire Wire Line
-	5325 2825 5475 2825
-Connection ~ 5475 2825
-Wire Wire Line
-	5475 2825 5475 3150
 $Comp
 L Connector_Generic:Conn_02x08_Odd_Even J123
@@
 Wire Wire Line
 	7800 6950 7900 6950
-Text GLabel 8500 6950 2    50   Output ~ 0
+Text GLabel 8875 7375 2    50   Output ~ 0
 OP
 Wire Wire Line
-	8400 6950 8500 6950
+	8775 7375 8875 7375
 Text GLabel 7800 6750 0    50   Input ~ 0
 RF_READY
 Wire Wire Line
 	7800 6750 7900 6750
-Text GLabel 8500 6750 2    50   Output ~ 0
+Text GLabel 9200 6950 2    50   Output ~ 0
 RESET_CMD
 Wire Wire Line
-	8400 6750 8500 6750
+	9100 6950 9200 6950
 Text GLabel 7800 6450 0    50   Input ~ 0
 ALC_MON
@@
 Wire Notes Line
 	9875 875  1275 875
+$Comp
+L Diode:BAT54CW D?
+U 1 1 5DEE2596
+P 8775 7175
+AR Path="/5E11E288/5DEE2596" Ref="D?"  Part="1"
+AR Path="/5DEE2596" Ref="D103"  Part="1"
+F 0 "D103" H 8425 7100 50  0000 L CNN
+F 1 "BAT54CW" H 8375 7000 50  0000 L CNN
+F 2 "Package_TO_SOT_SMD:SOT-323_SC-70" H 8850 7300 50  0001 L CNN
+F 3 "https://assets.nexperia.com/documents/data-sheet/BAT54W_SER.pdf" H 8695 7175 50  0001 C CNN
+	1    8775 7175
+	1    0    0    -1
+$EndComp
+Wire Wire Line
+	8400 7175 8475 7175
+Text GLabel 9125 7175 2    50   Input ~ 0
+OP_CMD_PI
+Wire Wire Line
+	9125 7175 9075 7175
+$Comp
+L Diode:BAT54CW D?
+U 1 1 5E035F59
+P 9100 6750
+AR Path="/5E11E288/5E035F59" Ref="D?"  Part="1"
+AR Path="/5E035F59" Ref="D104"  Part="1"
+F 0 "D104" H 8750 6675 50  0000 L CNN
+F 1 "BAT54CW" H 8700 6575 50  0000 L CNN
+F 2 "Package_TO_SOT_SMD:SOT-323_SC-70" H 9175 6875 50  0001 L CNN
+F 3 "https://assets.nexperia.com/documents/data-sheet/BAT54W_SER.pdf" H 9020 6750 50  0001 C CNN
+	1    9100 6750
+	1    0    0    -1
+$EndComp
+Text GLabel 9450 6750 2    50   Input ~ 0
+RESET_CMD_PI
+Wire Wire Line
+	9450 6750 9400 6750
+Wire Wire Line
+	8400 6750 8800 6750
+Wire Wire Line
+	8400 7175 8400 6950
+$Comp
+L Device:CP C?
+U 1 1 5DFBB614
+P 4100 2825
+AR Path="/5CBB0B33/5DFBB614" Ref="C?"  Part="1"
+AR Path="/5DFBB614" Ref="C105"  Part="1"
+F 0 "C105" H 4218 2871 50  0000 L CNN
+F 1 "47u" H 4218 2780 50  0000 L CNN
+F 2 "Capacitor_Tantalum_SMD:CP_EIA-6032-28_Kemet-C" H 4138 2675 50  0001 C CNN
+F 3 "~" H 4100 2825 50  0001 C CNN
+	1    4100 2825
+	1    0    0    -1
+$EndComp
+Wire Wire Line
+	3875 2525 4100 2525
+Wire Wire Line
+	3775 3125 4100 3125
+Wire Wire Line
+	4100 2675 4100 2525
+Connection ~ 4100 2525
+Wire Wire Line
+	4100 2525 4800 2525
+Wire Wire Line
+	4100 2975 4100 3125
+Connection ~ 4100 3125
+Wire Wire Line
+	4100 3125 4800 3125
+Wire Wire Line
+	5475 2150 5475 2825
+Wire Wire Line
+	5400 2825 5475 2825
+Connection ~ 5475 2825
+Wire Wire Line
+	5475 2825 5475 3150
+Wire Wire Line
+	4500 2825 4500 1950
+Wire Wire Line
+	4500 1950 5100 1950
 $EndSCHEMATC

Commit message: Review 2
Connections:
- net CONTROLLER/INT_OC is gone; now on net CONTROLLER/INT_OC: J107.4 (Pin_4)
- net CONTROLLER/INT_OC: no longer J121.4 (Pin_4)
- new net CONTROLLER/INT_OC: J121.4 (Pin_4)
Changed lines of the file:
@@
 EESchema Schematic File Version 4
-LIBS:RF-AMP-CNTLR_V1-cache
 EELAYER 30 0
 EELAYER END

Commit message: Review
Parts:
- C102, C103: value 470n -> 68n
- C104, C110, C111, C112, C113, C120, C121, C122: value 100u -> 47u
- C108, C109: value 470n -> 47n
- F101, F102: value 0.1AT -> 1AT
Connections:
- net CONTROLLER/INT_OC is gone; now on net CONTROLLER/INT_OC: J107.4 (Pin_4)
- net CONTROLLER/INT_OC: no longer J121.4 (Pin_4)
- new net CONTROLLER/INT_OC: J121.4 (Pin_4)
Other:
- moved on the sheet: C102, C103, FL101
Changed lines of the file:
@@
 Sheet 1 4
 Title "RF Amplifier Controller"
-Date "2019-12-01"
+Date "2020-01-19"
 Rev "1"
 Comp "HB9GKW"
@@
 AR Path="/5D99E420" Ref="C120"  Part="1"
 F 0 "C120" H 8418 1621 50  0000 L CNN
-F 1 "100u" H 8418 1530 50  0000 L CNN
+F 1 "47u" H 8418 1530 50  0000 L CNN
 F 2 "Capacitor_Tantalum_SMD:CP_EIA-6032-28_Kemet-C" H 8338 1425 50  0001 C CNN
 F 3 "~" H 8300 1575 50  0001 C CNN
@@
 L Device:EMI_Filter_CommonMode FL?
 U 1 1 5D99E459
-P 3300 1475
+P 3875 1475
 AR Path="/5CBB0B33/5D99E459" Ref="FL?"  Part="1"
 AR Path="/5D99E459" Ref="FL101"  Part="1"
-F 0 "FL101" H 3300 1662 50  0000 C CNN
-F 1 "EMI_Filter_CommonMode" H 3300 1662 50  0001 C CNN
-F 2 "Inductor_THT:Choke_Schaffner_RN202-04-8.8x18.2mm" V 3300 1515 50  0001 C CNN
-F 3 "~" V 3300 1515 50  0000 C CNN
-	1    3300 1475
+F 0 "FL101" H 3875 1662 50  0000 C CNN
+F 1 "EMI_Filter_CommonMode" H 3875 1662 50  0001 C CNN
+F 2 "Inductor_THT:Choke_Schaffner_RN202-04-8.8x18.2mm" V 3875 1515 50  0001 C CNN
+F 3 "~" V 3875 1515 50  0000 C CNN
+	1    3875 1475
 	1    0    0    -1
 $EndComp
@@
 L Device:C C?
 U 1 1 5D99E460
-P 3650 1475
+P 4325 1475
 AR Path="/5CBB0B33/5D99E460" Ref="C?"  Part="1"
 AR Path="/5D99E460" Ref="C103"  Part="1"
-F 0 "C103" H 3675 1550 50  0000 L CNN
-F 1 "470n" H 3675 1375 50  0000 L CNN
-F 2 "Capacitor_THT:C_Rect_L13.0mm_W4.0mm_P10.00mm_FKS3_FKP3_MKS4" H 3688 1325 50  0001 C CNN
-F 3 "~" H 3650 1475 50  0001 C CNN
-	1    3650 1475
+F 0 "C103" H 4425 1525 50  0000 L CNN
+F 1 "68n" H 4425 1425 50  0000 L CNN
+F 2 "Capacitor_THT:C_Rect_L13.0mm_W4.0mm_P10.00mm_FKS3_FKP3_MKS4" H 4363 1325 50  0001 C CNN
+F 3 "~" H 4325 1475 50  0001 C CNN
+	1    4325 1475
 	1    0    0    -1
 $EndComp
@@
 L Device:C C?
 U 1 1 5D99E469
-P 2925 1475
+P 3425 1475
 AR Path="/5CBB0B33/5D99E469" Ref="C?"  Part="1"
 AR Path="/5D99E469" Ref="C102"  Part="1"
-F 0 "C102" H 2700 1550 50  0000 L CNN
-F 1 "470n" H 2725 1375 50  0000 L CNN
-F 2 "Capacitor_THT:C_Rect_L13.0mm_W4.0mm_P10.00mm_FKS3_FKP3_MKS4" H 2963 1325 50  0001 C CNN
-F 3 "~" H 2925 1475 50  0001 C CNN
-	1    2925 1475
+F 0 "C102" H 3125 1525 50  0000 L CNN
+F 1 "68n" H 3175 1425 50  0000 L CNN
+F 2 "Capacitor_THT:C_Rect_L13.0mm_W4.0mm_P10.00mm_FKS3_FKP3_MKS4" H 3463 1325 50  0001 C CNN
+F 3 "~" H 3425 1475 50  0001 C CNN
+	1    3425 1475
 	1    0    0    -1
 $EndComp
@@
 AR Path="/5D99E506" Ref="F101"  Part="1"
 F 0 "F101" V 2103 1250 50  0000 C CNN
-F 1 "0.1AT" V 2194 1250 50  0000 C CNN
+F 1 "1AT" V 2194 1250 50  0000 C CNN
 F 2 "Fuse:Fuse_Littelfuse_372_D8.50mm" V 2230 1250 50  0001 C CNN
 F 3 "~" H 2300 1250 50  0001 C CNN
@@
 AR Path="/5D99E50D" Ref="F102"  Part="1"
 F 0 "F102" V 2400 1350 50  0000 C CNN
-F 1 "0.1AT" V 2475 1350 50  0000 C CNN
+F 1 "1AT" V 2475 1350 50  0000 C CNN
 F 2 "Fuse:Fuse_Littelfuse_372_D8.50mm" V 2230 1350 50  0001 C CNN
 F 3 "~" H 2300 1350 50  0001 C CNN
@@
 $EndComp
 Wire Wire Line
-	3100 1575 3100 1700
-Wire Wire Line
-	3100 1250 3100 1375
-Wire Wire Line
-	2925 1325 2925 1250
-Wire Wire Line
-	2925 1250 3100 1250
-Wire Wire Line
-	2925 1625 2925 1700
-Wire Wire Line
-	2925 1700 3100 1700
-Wire Wire Line
-	3500 1700 3650 1700
-Wire Wire Line
-	3500 1250 3650 1250
+	3675 1575 3675 1700
+Wire Wire Line
+	3675 1250 3675 1375
+Wire Wire Line
+	3425 1325 3425 1250
+Wire Wire Line
+	3425 1250 3675 1250
+Wire Wire Line
+	3425 1625 3425 1700
+Wire Wire Line
+	3425 1700 3675 1700
+Wire Wire Line
+	4075 1700 4325 1700
+Wire Wire Line
+	4075 1250 4325 1250
 Wire Wire Line
 	5800 1575 5800 1700
@@
 	5800 1250 5800 1375
 Wire Wire Line
-	3500 1250 3500 1375
-Wire Wire Line
-	3500 1575 3500 1700
-Wire Wire Line
-	3650 1625 3650 1700
+	4075 1250 4075 1375
+Wire Wire Line
+	4075 1575 4075 1700
+Wire Wire Line
+	4325 1625 4325 1700
 Connection ~ 5475 1700
 Wire Wire Line
 	5475 1700 5800 1700
 Wire Wire Line
-	3650 1325 3650 1250
+	4325 1325 4325 1250
 $Comp
 L Connector:Screw_Terminal_01x06 J?
@@
 AR Path="/5CBB0B33/5D3E9E7E" Ref="C?"  Part="1"
 AR Path="/5D3E9E7E" Ref="C111"  Part="1"
-F 0 "C111" H 6825 1650 50  0000 L CNN
-F 1 "100u" H 6850 1500 50  0000 L CNN
+F 0 "C111" H 6800 1625 50  0000 L CNN
+F 1 "47u" H 6850 1525 50  0000 L CNN
 F 2 "Capacitor_Tantalum_SMD:CP_EIA-6032-28_Kemet-C" H 7138 1425 50  0001 C CNN
 F 3 "~" H 7100 1575 50  0001 C CNN
@@
 AR Path="/5D3F9EE7" Ref="C121"  Part="1"
 F 0 "C121" H 7975 2300 50  0000 L CNN
-F 1 "100u" H 7975 2400 50  0000 L CNN
+F 1 "47u" H 8025 2400 50  0000 L CNN
 F 2 "Capacitor_Tantalum_SMD:CP_EIA-6032-28_Kemet-C" H 8338 2200 50  0001 C CNN
 F 3 "~" H 8300 2350 50  0001 C CNN
@@
 AR Path="/5CBB0B33/5D3F9F1D" Ref="C?"  Part="1"
 AR Path="/5D3F9F1D" Ref="C112"  Part="1"
-F 0 "C112" H 7250 2275 50  0000 L CNN
-F 1 "100u" H 7175 2425 50  0000 L CNN
+F 0 "C112" H 7225 2300 50  0000 L CNN
+F 1 "47u" H 7225 2400 50  0000 L CNN
 F 2 "Capacitor_Tantalum_SMD:CP_EIA-6032-28_Kemet-C" H 7138 2200 50  0001 C CNN
 F 3 "~" H 7100 2350 50  0001 C CNN
@@
 AR Path="/5D586DF5" Ref="C122"  Part="1"
 F 0 "C122" H 8418 3196 50  0000 L CNN
-F 1 "100u" H 8418 3105 50  0000 L CNN
+F 1 "47u" H 8418 3105 50  0000 L CNN
 F 2 "Capacitor_Tantalum_SMD:CP_EIA-6032-28_Kemet-C" H 8338 3000 50  0001 C CNN
 F 3 "~" H 8300 3150 50  0001 C CNN
@@
 AR Path="/5D586E2A" Ref="C113"  Part="1"
 F 0 "C113" H 6825 3225 50  0000 L CNN
-F 1 "100u" H 6850 3075 50  0000 L CNN
+F 1 "47u" H 6850 3075 50  0000 L CNN
 F 2 "Capacitor_Tantalum_SMD:CP_EIA-6032-28_Kemet-C" H 7138 3000 50  0001 C CNN
 F 3 "~" H 7100 3150 50  0001 C CNN
@@
 	1    0    0    -1
 $EndComp
-Connection ~ 3650 1250
-Connection ~ 3650 1700
-Wire Wire Line
-	3650 1250 5675 1250
+Connection ~ 4325 1250
+Connection ~ 4325 1700
+Wire Wire Line
+	4325 1250 5675 1250
 $Comp
 L Converter_DCDC:ITQ2412SA PS104
@@
 AR Path="/5D59BBDE" Ref="C110"  Part="1"
 F 0 "C110" H 5593 4371 50  0000 L CNN
-F 1 "100u" H 5593 4280 50  0000 L CNN
+F 1 "47u" H 5593 4280 50  0000 L CNN
 F 2 "Capacitor_Tantalum_SMD:CP_EIA-6032-28_Kemet-C" H 5513 4175 50  0001 C CNN
 F 3 "~" H 5475 4325 50  0001 C CNN
@@
 AR Path="/5D59BC11" Ref="C104"  Part="1"
 F 0 "C104" H 3975 4425 50  0000 L CNN
-F 1 "100u" H 4000 4250 50  0000 L CNN
+F 1 "47u" H 4000 4250 50  0000 L CNN
 F 2 "Capacitor_Tantalum_SMD:CP_EIA-6032-28_Kemet-C" H 4288 4175 50  0001 C CNN
 F 3 "~" H 4250 4325 50  0001 C CNN
@@
 AR Path="/5D83FED4" Ref="C109"  Part="1"
 F 0 "C109" V 5100 2750 50  0000 L CNN
-F 1 "470n" V 5400 2750 50  0000 L CNN
+F 1 "47n" V 5400 2750 50  0000 L CNN
 F 2 "Capacitor_THT:C_Rect_L7.0mm_W3.5mm_P5.00mm" H 5288 2675 50  0001 C CNN
 F 3 "~" H 5250 2825 50  0001 C CNN
@@
 $EndComp
 Wire Wire Line
-	3650 1700 5475 1700
+	4325 1700 5475 1700
 $Comp
 L Device:C C?
@@
 AR Path="/5D902ABA" Ref="C108"  Part="1"
 F 0 "C108" V 5100 1875 50  0000 L CNN
-F 1 "470n" V 5400 1875 50  0000 L CNN
+F 1 "47n" V 5400 1875 50  0000 L CNN
 F 2 "Capacitor_THT:C_Rect_L7.0mm_W3.5mm_P5.00mm" H 5288 1800 50  0001 C CNN
 F 3 "~" H 5250 1950 50  0001 C CNN
@@
 AR Path="/5CBB0B33/5D98C37C" Ref="R?"  Part="1"
 AR Path="/5D98C37C" Ref="R101"  Part="1"
-F 0 "R101" V 2600 2825 50  0000 L CNN
-F 1 "22k" V 2675 2850 50  0000 L CNN
+F 0 "R101" V 2625 2825 50  0000 L CNN
+F 1 "22k" V 2700 2850 50  0000 L CNN
 F 2 "Resistor_SMD:R_0805_2012Metric_Pad1.15x1.40mm_HandSolder" V 2705 2925 50  0001 C CNN
 F 3 "~" H 2775 2925 50  0001 C CNN
@@
 AR Path="/5CBB0B33/5DA2786A" Ref="R?"  Part="1"
 AR Path="/5DA2786A" Ref="R102"  Part="1"
-F 0 "R102" V 3200 3625 50  0000 L CNN
-F 1 "1k" V 3275 3650 50  0000 L CNN
+F 0 "R102" V 3225 3625 50  0000 L CNN
+F 1 "1k" V 3300 3675 50  0000 L CNN
 F 2 "Resistor_SMD:R_0805_2012Metric_Pad1.15x1.40mm_HandSolder" V 3305 3725 50  0001 C CNN
 F 3 "~" H 3375 3725 50  0001 C CNN
@@
 Wire Wire Line
 	2450 1250 2625 1250
-Connection ~ 2925 1250
+Connection ~ 3425 1250
 Wire Wire Line
 	2075 1550 2625 1550
@@
 Connection ~ 2625 1250
 Wire Wire Line
-	2625 1250 2925 1250
+	2625 1250 3425 1250
 Wire Wire Line
 	2500 1650 2500 1700
 Wire Wire Line
-	2500 1700 2925 1700
+	2500 1700 3425 1700
 Connection ~ 2500 1650
-Connection ~ 2925 1700
+Connection ~ 3425 1700
 Wire Wire Line
 	4625 6025 4800 6025
