File: FRONTEND.sch (KiCad schematic (older format))
At the start: 182 parts, among them Q1 BC857, Q10 BCX53, Q11 BCX53, Q12 BCX53, Q2 IXTH140P10T, Q3 DTC124E, Q4 IXTH140P10T, Q5 DTA124E, Q6 DTC124E, Q7 DTC124E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

Commit message: ALC latch-up fix
Parts:
- added D19: BZT52C4V7T-7, Diode_SMD:D_SOD-123, symbol Diode:DZ2S047X0L
- added R103: 4k7, Resistor_SMD:R_0805_2012Metric_Pad1.15x1.40mm_HandSolder, symbol Device:R
- R10: value 100k -> 68k
- R73: value 100k -> 470
Connections:
- net -12V: now also R103.2; no longer Q6.2 (E)
- net Earth: now also D19.1 (K)
- net FWD4_MON: no longer R57.2
- new net: D19.2 (A), Q6.2 (E), R103.1
- new net FWD: R57.2
Other:
- moved on the sheet: Q5, Q6
Changed lines of the file:
@@
 Sheet 2 3
 Title "RF Amplifier Controller"
-Date "2020-07-24"
+Date "2020-10-25"
 Rev "1"
 Comp "HB9GKW"
@@
 AR Path="/5E11E288/5F9D3583" Ref="R73"  Part="1"
 F 0 "R73" V 10425 9325 50  0000 R CNN
-F 1 "100k" V 10350 9350 50  0000 R CNN
+F 1 "470" V 10350 9325 50  0000 R CNN
 F 2 "Resistor_SMD:R_0805_2012Metric_Pad1.15x1.40mm_HandSolder" V 10455 9250 50  0001 C CNN
 F 3 "~" H 10525 9250 50  0001 C CNN
@@
 AR Path="/5E11E288/620D23DD" Ref="R10"  Part="1"
 F 0 "R10" V 2425 3700 50  0000 R CNN
-F 1 "100k" V 2350 3725 50  0000 R CNN
+F 1 "68k" V 2350 3700 50  0000 R CNN
 F 2 "Resistor_SMD:R_0805_2012Metric_Pad1.15x1.40mm_HandSolder" V 2205 3625 50  0001 C CNN
 F 3 "~" H 2275 3625 50  0001 C CNN
@@
 Connection ~ 10825 1375
 Wire Wire Line
-	9325 1275 9925 1275
-Connection ~ 9925 1275
-Wire Wire Line
-	9925 1275 10175 1275
-Wire Wire Line
 	8925 1275 9025 1275
 Wire Wire Line
@@
 Text HLabel 11700 1375 2    50   Output ~ 0
 ALC
-Text HLabel 7650 1375 0    50   Input ~ 0
-FWD4_MON
 $Comp
 L Device:C C?
@@
 $EndComp
 Wire Wire Line
-	9925 1275 9925 2075
+	10000 1275 10000 1500
 $Comp
 L Transistor_BJT:DTC124E Q6
 U 1 1 621E821C
-P 9825 2275
+P 9900 1700
 AR Path="/5E11E288/621E821C" Ref="Q6"  Part="1"
 AR Path="/5D2BEC5D/621E821C" Ref="Q?"  Part="1"
-F 0 "Q6" H 10000 2300 50  0000 L CNN
-F 1 "DTC124E" H 10000 2225 50  0000 L CNN
-F 2 "Package_TO_SOT_SMD:SOT-23" H 9825 2275 50  0001 L CNN
-F 3 "" H 9825 2275 50  0001 L CNN
-	1    9825 2275
+F 0 "Q6" H 9825 1975 50  0000 L CNN
+F 1 "DTC124E" H 9650 1900 50  0000 L CNN
+F 2 "Package_TO_SOT_SMD:SOT-23" H 9900 1700 50  0001 L CNN
+F 3 "" H 9900 1700 50  0001 L CNN
+	1    9900 1700
 	1    0    0    -1
 $EndComp
@@
 L power:-12V #PWR?
 U 1 1 621E8203
-P 9925 2475
+P 10000 2375
 AR Path="/5D2BEC5D/621E8203" Ref="#PWR?"  Part="1"
 AR Path="/5E11E288/621E8203" Ref="#PWR0145"  Part="1"
-F 0 "#PWR0145" H 9925 2575 50  0001 C CNN
-F 1 "-12V" H 9940 2648 50  0000 C CNN
-F 2 "" H 9925 2475 50  0001 C CNN
-F 3 "" H 9925 2475 50  0001 C CNN
-	1    9925 2475
+F 0 "#PWR0145" H 10000 2475 50  0001 C CNN
+F 1 "-12V" H 10015 2548 50  0000 C CNN
+F 2 "" H 10000 2375 50  0001 C CNN
+F 3 "" H 10000 2375 50  0001 C CNN
+	1    10000 2375
 	1    0    0    1
 $EndComp
@@
 L power:+5V #PWR?
 U 1 1 613D66DB
-P 9500 1875
+P 9175 1625
 AR Path="/5CBD59C6/613D66DB" Ref="#PWR?"  Part="1"
 AR Path="/5D2BEC5D/613D66DB" Ref="#PWR?"  Part="1"
 AR Path="/5E11E288/613D66DB" Ref="#PWR0144"  Part="1"
-F 0 "#PWR0144" H 9500 1725 50  0001 C CNN
-F 1 "+5V" H 9515 2048 50  0000 C CNN
-F 2 "" H 9500 1875 50  0001 C CNN
-F 3 "" H 9500 1875 50  0001 C CNN
-	1    9500 1875
+F 0 "#PWR0144" H 9175 1475 50  0001 C CNN
+F 1 "+5V" H 9190 1798 50  0000 C CNN
+F 2 "" H 9175 1625 50  0001 C CNN
+F 3 "" H 9175 1625 50  0001 C CNN
+	1    9175 1625
 	1    0    0    -1
 $EndComp
-Wire Wire Line
-	9500 2275 9575 2275
 $Comp
 L Transistor_BJT:DTA124E Q5
 U 1 1 621E8236
-P 9400 2075
+P 9450 1800
 AR Path="/5E11E288/621E8236" Ref="Q5"  Part="1"
 AR Path="/621E8236" Ref="Q?"  Part="1"
 AR Path="/5D2BEC5D/621E8236" Ref="Q?"  Part="1"
-F 0 "Q5" H 9150 1825 50  0000 C CNN
-F 1 "DTA124E" H 9250 1900 50  0000 C CNN
-F 2 "Package_TO_SOT_SMD:SOT-23" H 9400 2075 50  0001 L CNN
-F 3 "" H 9400 2075 50  0001 L CNN
-	1    9400 2075
-	1    0    0    1
+F 0 "Q5" V 9750 1800 50  0000 C CNN
+F 1 "DTA124E" V 9675 1800 50  0000 C CNN
+F 2 "Package_TO_SOT_SMD:SOT-23" H 9450 1800 50  0001 L CNN
+F 3 "" H 9450 1800 50  0001 L CNN
+	1    9450 1800
+	0    1    -1   0
 $EndComp
-Wire Wire Line
-	9100 2075 9150 2075
-Text HLabel 9100 2075 0    50   Input ~ 0
+Text HLabel 9375 2125 0    50   Input ~ 0
 GATE_ALC_EN
 $Comp
@@
 	1    0    0    1
 $EndComp
+Connection ~ 10000 1275
+Wire Wire Line
+	10000 1275 10175 1275
+Wire Wire Line
+	9325 1275 10000 1275
+Wire Wire Line
+	9175 1625 9175 1700
+Wire Wire Line
+	9175 1700 9250 1700
+Wire Wire Line
+	9375 2125 9450 2125
+Wire Wire Line
+	9450 2125 9450 2050
+$Comp
+L Diode:DZ2S047X0L D19
+U 1 1 5FD3E99D
+P 10225 2000
+AR Path="/5E11E288/5FD3E99D" Ref="D19"  Part="1"
+AR Path="/5D2BEC5D/5FD3E99D" Ref="D?"  Part="1"
+F 0 "D19" H 10175 1825 50  0000 L CNN
+F 1 "BZT52C4V7T-7" H 9800 1900 50  0000 L CNN
+F 2 "Diode_SMD:D_SOD-123" H 10225 1825 50  0001 C CNN
+F 3 "https://www.mouser.ch/datasheet/2/115/ds30502-1142513.pdf" H 10225 2000 50  0001 C CNN
+	1    10225 2000
+	-1   0    0    1
+$EndComp
+$Comp
+L Device:R R?
+U 1 1 5FE84A8C
+P 10000 2225
+AR Path="/5FE84A8C" Ref="R?"  Part="1"
+AR Path="/5C000D65/5FE84A8C" Ref="R?"  Part="1"
+AR Path="/5E11E288/5FE84A8C" Ref="R103"  Part="1"
+F 0 "R103" V 10150 2300 50  0000 R CNN
+F 1 "4k7" V 10075 2300 50  0000 R CNN
+F 2 "Resistor_SMD:R_0805_2012Metric_Pad1.15x1.40mm_HandSolder" V 9930 2225 50  0001 C CNN
+F 3 "~" H 10000 2225 50  0001 C CNN
+	1    10000 2225
+	-1   0    0    -1
+$EndComp
+Wire Wire Line
+	10000 1900 10000 2000
+Wire Wire Line
+	10000 2000 10075 2000
+Connection ~ 10000 2000
+Wire Wire Line
+	10000 2000 10000 2075
+$Comp
+L power:Earth #PWR?
+U 1 1 6000C197
+P 10450 2075
+AR Path="/6000C197" Ref="#PWR?"  Part="1"
+AR Path="/5C000D65/6000C197" Ref="#PWR?"  Part="1"
+AR Path="/5D2BEC5D/6000C197" Ref="#PWR?"  Part="1"
+AR Path="/5E11E288/6000C197" Ref="#PWR0275"  Part="1"
+F 0 "#PWR0275" H 10450 1825 50  0001 C CNN
+F 1 "Earth" H 10450 1925 50  0001 C CNN
+F 2 "" H 10450 2075 50  0001 C CNN
+F 3 "" H 10450 2075 50  0001 C CNN
+	1    10450 2075
+	1    0    0    -1
+$EndComp
+Wire Wire Line
+	10375 2000 10450 2000
+Wire Wire Line
+	10450 2000 10450 2075
+Text GLabel 7650 1375 0    50   Input ~ 0
+FWD
 $EndSCHEMATC
